Commit message: 阶段 0-5：腿改 revolute、六执行器链路、离线 A/B 生成、全身 Pitch/Roll LQR 与安全分配
- 阶段 0：四个腿关节 fixed → revolute（轴 y、零位即标准姿态、限位/力矩抄模型），轮径统一 0.030
- 阶段 1：六执行器链路（六路桥接 + 六个 MotorNode + 四段腿参数 + /joint_states 六关节解析）
- 阶段 2：腿姿保持器（静态重力前馈 U0 + PD；标准姿态 U0 = 胯 -0.0147 / 膝 -0.2567 N·m）
- 阶段 3/4：离线工具 tools/generate_wheel_leg_lqr（展开 URDF → 平面共模 8 状态 Pitch、前视面 4 状态 Roll → X0/U0/A/B/K → 增益文件，21 项检查）
- 阶段 5：TorqueAllocator（共模优先、左右成组限幅与变化率、髋膝软限位、NaN 清零）+ 联合安全状态机（反馈超时 / 姿态 / 越界 / 周期），带消融开关与单元测试
- 键盘：framework 层只加 '=' / '-' 键检测，不持有机器人数据
- 世界：加梯形障碍（车高一半 ≈ 60 mm、15° 缓坡）
- 文档：实施规划、平面模型参数与公式、当前状态与节点职责

Co-Authored-By: Claude Code <noreply@anthropic.com>

File: project/robot/models/bodys/wheel_leg_robot.xacro (robot description, xacro)
@@ -4,5 +4,5 @@
      坐标系约定（`ros2 run xacro` 或 spawn 的时候按这个来）：
        base_link 原点是整车参考点，摆在**轮轴高度**上 —— 所以两个轮子的关节 z 都是 0，
-       整车 spawn 的 z 就填轮子半径（0.04），两个轮子正好同时贴地。
+       整车 spawn 的 z 就填轮子半径（0.03），两个轮子正好同时贴地。
      竖直方向（都是从轮轴那一层往上量）：
        胯轴 / 大腿根 = 2·leg_drop = 72mm（腿在标准姿态下把车身顶到这么高）
@@ -13,7 +13,9 @@
      横向：胯/腿在 y = ±38mm；轮子还要再往外 22mm（外侧 y = ±60mm），
      所以轮子内侧离底盘侧面 5mm，跟四轮车那边一样。
-     标准姿态：α = 40°，两条腿都不动 —— 胯关节、膝关节、腿的固定关节现在**全是 fixed**，
-     只有轮子是 continuous（驱动轮，力矩电机插件由 wheel 宏自己挂）。
-     要让它能伸缩，见 modules/leg.xacro 顶上那段（改成 revolute 的位置和取值都写在那儿）。
+     标准姿态：α = 40°（与水平面，也就是文件头说的竖直方向 72mm）。
+     六个运动关节：左右胯、左右膝是 **revolute**（绕 y，力矩入口由 leg 宏挂的 torque_motor 给），
+     左右轮是 continuous（驱动轮）。胯/膝那两个枢轴圆柱只是装饰，仍然是 fixed。
+     腿的符号约定、限位、关节力矩见 modules/leg.xacro 顶上那段；
+     现在还没有腿姿保持器（文档 §8 阶段 2），所以跑起来腿会在自重下折下去。
      反馈与 IMU：
        joint_encoder 是**模型级**插件（一个模型挂一次，不是每个关节一次），
@@ -48,5 +50,6 @@
     joint_name="left_hip_joint"
     parent="base_link"
-    xyz="0 ${leg_y_offset} ${hip_height}"/>
+    xyz="0 ${leg_y_offset} ${hip_height}"
+    lower="${hip_limit_lower}" upper="${hip_limit_upper}"/>
   <!-- 膝盖圆柱在大腿远端 -->
   <xacro:knee name="left_knee_link"
@@ -58,5 +61,6 @@
     joint_name="left_knee_joint"
     parent="left_knee_link"
-    direction="-1"/>
+    direction="-1"
+    lower="${knee_limit_lower}" upper="${knee_limit_upper}"/>
   <!-- 轮子在小腿远端。y 要再往外挪 (轮距/2 - 腿侧偏)：腿在 38mm、轮子在 60mm -->
   <xacro:wheel name="left_wheel_link"
@@ -72,5 +76,6 @@
     joint_name="right_hip_joint"
     parent="base_link"
-    xyz="0 ${-leg_y_offset} ${hip_height}"/>
+    xyz="0 ${-leg_y_offset} ${hip_height}"
+    lower="${hip_limit_lower}" upper="${hip_limit_upper}"/>
   <xacro:knee name="right_knee_link"
     joint_name="right_knee_cylinder_joint"
@@ -80,5 +85,6 @@
     joint_name="right_knee_joint"
     parent="right_knee_link"
-    direction="-1"/>
+    direction="-1"
+    lower="${knee_limit_lower}" upper="${knee_limit_upper}"/>
   <xacro:wheel name="right_wheel_link"
     joint_name="right_wheel_joint"

File: project/robot/models/modules/hip.xacro (robot description, xacro)
@@ -12,4 +12,5 @@
 <robot xmlns:xacro="http://www.ros.org/wiki/xacro">
   <xacro:include filename="$(find gazebo)/models/basic/cylinder.xacro"/>
+  <xacro:include filename="$(find gazebo)/models/basic/joint.xacro"/>
   <xacro:macro name="hip" params="
     name
@@ -30,5 +31,5 @@
       radius="${radius}"
       length="${width}"
-      rpy="1.57079632679 0 0"
+      rpy="${90.0 * pi / 180.0} 0 0"
       mass="${mass}"
       ixx="${ixx}"
@@ -37,9 +38,5 @@
       color_name="${color_name}"
       color_rgba="${color_rgba}"/>
-    <joint name="${joint_name}" type="fixed">
-      <parent link="${parent}"/>
-      <child link="${name}"/>
-      <origin xyz="${xyz}" rpy="0 0 0"/>
-    </joint>
+    <xacro:fixed_joint name="${joint_name}" parent="${parent}" child="${name}" xyz="${xyz}"/>
   </xacro:macro>
 </robot>

File: project/robot/models/modules/knee.xacro (robot description, xacro)
@@ -13,4 +13,5 @@
 <robot xmlns:xacro="http://www.ros.org/wiki/xacro">
   <xacro:include filename="$(find gazebo)/models/basic/cylinder.xacro"/>
+  <xacro:include filename="$(find gazebo)/models/basic/joint.xacro"/>
   <xacro:macro name="knee" params="
     name
@@ -30,5 +31,5 @@
       radius="${radius}"
       length="${width}"
-      rpy="1.57079632679 0 0"
+      rpy="${90.0 * pi / 180.0} 0 0"
       mass="${mass}"
       ixx="${ixx}"
@@ -37,9 +38,5 @@
       color_name="${color_name}"
       color_rgba="${color_rgba}"/>
-    <joint name="${joint_name}" type="fixed">
-      <parent link="${parent}"/>
-      <child link="${name}"/>
-      <origin xyz="${xyz}" rpy="0 0 0"/>
-    </joint>
+    <xacro:fixed_joint name="${joint_name}" parent="${parent}" child="${name}" xyz="${xyz}"/>
   </xacro:macro>
 </robot>

File: project/robot/models/modules/leg.xacro (robot description, xacro)
@@ -13,17 +13,30 @@
        +1 → 远端在 ( +leg_span, 0, -leg_drop )，往前下方（大腿）
        -1 → 远端在 ( -leg_span, 0, -leg_drop )，往后下方（小腿）
-     标准姿态就是这套默认值（α = 40°），腿现在**不动**：关节写死 fixed。
-     以后要伸缩，把下面的 fixed 换成 revolute 并补 limit —— lqr 那边的取值是
-     effort 1.5 N·m、velocity 6.0 rad/s、damping 0.05；符号约定 α = 50° - q_hip、
-     β = 80° - q_knee，对称伸缩（e = 0）时 q_knee = -2·q_hip。
-     用法（在 body 里）：
+     标准姿态就是这套默认值（α = 40°）。
+     关节是 **revolute**（绕 y），q = 0 就是上面这个标准姿态（α=50°、β=80°、胯到轮轴 72mm）——
+     关节原点不转、几何体按标准姿态画，所以零位天然对上。符号跟 lqr 那台的
+     leg_wheel_robot.urdf.xacro 完全一致（那边的 q_urdf_hip 就是这里的 q_hip）：
+       α = 50° - q_hip（α 从**竖直**量）、β = 80° - q_knee（膝内角，从伸直量），
+       对称伸缩（e = 0，轮子还在胯轴正下方）时 q_knee = -2·q_hip；
+       q_hip > 0 = 腿伸直、车身变高。
+       限位不对称（胯 [-15°, 35°]、膝 [-65°, 25°]），按对称伸缩走实际只到
+       q_hip ∈ [-12.5°, +32.5°]（先顶到膝的 -65°，不是胯自己的 [-15°, +35°]）；
+       关节力矩 1.5 N·m（静态需求约 3 倍余量）、转速 6.0 rad/s、阻尼 0.05。
+     力矩入口：每个腿关节挂一个 torque_motor，跟轮子同一个插件，话题
+     /model/<模型名>/joint/<关节名>/cmd_force。现在没人往里发力矩（腿姿保持器见文档 §8 阶段 2），
+     所以**光跑仿真腿会在自重下折下去**，不是模型改错了。
+     用法（在 body 里，限位按关节传 leg.xacro 顶上那几个 property）：
        <xacro:leg name="left_thigh_link" joint_name="left_hip_joint"
-                  parent="base_link"           xyz="0 ${leg_y_offset} ${hip_height}"/>
+                  parent="base_link" xyz="0 ${leg_y_offset} ${hip_height}"
+                  lower="${hip_limit_lower}"  upper="${hip_limit_upper}"/>
        <xacro:leg name="left_calf_link"  joint_name="left_knee_joint"
-                  parent="left_knee_link"      direction="-1"/> -->
+                  parent="left_knee_link" direction="-1"
+                  lower="${knee_limit_lower}" upper="${knee_limit_upper}"/> -->
 <robot xmlns:xacro="http://www.ros.org/wiki/xacro">
   <xacro:include filename="$(find gazebo)/models/basic/box.xacro"/>
+  <xacro:include filename="$(find gazebo)/models/basic/joint.xacro"/>
+  <xacro:include filename="$(find gazebo)/plugins/motor/torque_motor.xacro"/>
   <xacro:property name="leg_length"    value="0.056"/>
-  <xacro:property name="leg_angle"     value="0.6981317008"/>
+  <xacro:property name="leg_angle"     value="${40.0 * pi / 180.0}"/>
   <xacro:property name="leg_span"      value="${leg_length * cos(leg_angle)}"/>
   <xacro:property name="leg_drop"      value="${leg_length * sin(leg_angle)}"/>
@@ -31,10 +44,21 @@
   <xacro:property name="leg_half_drop" value="${leg_drop * 0.5}"/>
   <xacro:property name="leg_pitch"     value="${pi / 2 - leg_angle}"/>
+  <!-- 胯/膝的行程（详见文件头）。软限位是控制器里的事，这里写的是硬限位 -->
+  <xacro:property name="hip_limit_lower"  value="${-15.0 * pi / 180.0}"/>
+  <xacro:property name="hip_limit_upper"  value="${ 35.0 * pi / 180.0}"/>
+  <xacro:property name="knee_limit_lower" value="${-65.0 * pi / 180.0}"/>
+  <xacro:property name="knee_limit_upper" value="${ 25.0 * pi / 180.0}"/>
+  <xacro:property name="leg_effort"       value="1.5"/>
+  <xacro:property name="leg_velocity"     value="6.0"/>
+  <xacro:property name="leg_damping"      value="0.05"/>
   <xacro:macro name="leg" params="
     name
     joint_name
     parent
+    lower
+    upper
     xyz:='0 0 0'
     direction:=1
+    motor:='true'
     section:='0.016 0.018'
     mass:=0.03
@@ -59,9 +83,11 @@
       color_name="${color_name}"
       color_rgba="${color_rgba}"/>
-    <joint name="${joint_name}" type="fixed">
-      <parent link="${parent}"/>
-      <child link="${name}"/>
-      <origin xyz="${xyz}" rpy="0 0 0"/>
-    </joint>
+    <!-- 绕 y：整台车的关节都躺在 y 轴上，轴向量传错不报错，只是模型静默地转错方向 -->
+    <xacro:revolute_joint name="${joint_name}" parent="${parent}" child="${name}" xyz="${xyz}"
+                          lower="${lower}" upper="${upper}"
+                          effort="${leg_effort}" velocity="${leg_velocity}" damping="${leg_damping}"/>
+    <xacro:if value="${motor}">
+      <xacro:torque_motor joint_name="${joint_name}"/>
+    </xacro:if>
   </xacro:macro>
 </robot>

File: project/robot/models/modules/wheel.xacro (robot description, xacro)
@@ -1,6 +1,6 @@
 <?xml version="1.0"?>
-<!-- 轮子：尺寸是定死的 —— 半径 40mm、宽 20mm、0.15kg，跟 lqr 那台整机上的同名轮子一模一样。
+<!-- 轮子：尺寸是定死的 —— 半径 30mm、宽 15mm、0.15kg（宏参数里那两个默认值就是它，body 不覆盖）。
      为什么要转 90°：cylinder_link 出来的圆柱默认轴沿 z，轮子的轴得沿 y，
-     所以 visual / inertial / collision 统一 rpy="1.57 0 0" 躺倒，关节也绕 y 转。
+     所以 visual / inertial / collision 统一 rpy="${90.0 * pi / 180.0} 0 0" 躺倒，关节也绕 y 转。
      这样关节正转才是"往前滚"，LQR 那边算出来的力矩符号才对得上。
      电机：轮子是驱动轮，默认就把力矩电机插件（gz 的 ApplyJointForce）挂在自己的关节上，
@@ -22,4 +22,5 @@
   <xacro:include filename="$(find gazebo)/models/basic/cylinder.xacro"/>
   <xacro:include filename="$(find gazebo)/plugins/motor/torque_motor.xacro"/>
+  <xacro:include filename="$(find gazebo)/models/basic/joint.xacro"/>
   <xacro:macro name="wheel" params="
     name
@@ -44,5 +45,5 @@
       radius="${radius}"
       length="${width}"
-      rpy="1.57079632679 0 0"
+      rpy="${90.0 * pi / 180.0} 0 0"
       mass="${mass}"
       ixx="${ixx}"
@@ -51,11 +52,6 @@
       color_name="${color_name}"
       color_rgba="${color_rgba}"/>
-    <joint name="${joint_name}" type="continuous">
-      <parent link="${parent}"/>
-      <child link="${name}"/>
-      <origin xyz="${xyz}" rpy="0 0 0"/>
-      <axis xyz="0 1 0"/>
-      <limit effort="${effort}" velocity="${velocity}"/>
-    </joint>
+    <xacro:continuous_joint name="${joint_name}" parent="${parent}" child="${name}" xyz="${xyz}"
+                            effort="${effort}" velocity="${velocity}"/>
     <!-- 摩擦：必须各向异性，不然车只能直着走、转不了弯。
          四个轮子都是固定轮（没有转向关节），转向靠左右轮速差，那是要四个轮子横着刮地的。
